File: LTE-alarm-hw/LTE-alarm-hw.kicad_sch (KiCad schematic)
At the start: 14 parts, among them J1 ADXL345_I2C, J2 RELAY_0, J3 RELAY_1, J4 RELAY_2, Q1 AO3400A, SW1 SW_Push, SW2 SW_Push

Commit message: URL with SMS
Connections:
- net BUTTON0: now also A1.24 (D9); no longer A1.9 (A0)
- net BUTTON1: now also A1.25 (D10); no longer A1.10 (A1)
- net VDD: no longer J1.2 (Pin_2)
- net +3.3V: now reaches A1.4 (3V3)
- net +3.3V: now also J1.2 (Pin_2)
- no-connect marks 20 -> 19
Changed lines of the file:
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@@
   (no_connect (at 127 81.28))
   (no_connect (at 152.4 101.6))
-  (no_connect (at 127 101.6))
   (no_connect (at 127 96.52))
+  (no_connect (at 152.4 93.98))
   (no_connect (at 152.4 78.74))
-  (no_connect (at 142.24 68.58))
   (no_connect (at 218.44 64.77))
+  (no_connect (at 152.4 96.52))
   (no_connect (at 127 109.22))
   (no_connect (at 218.44 59.69))
   (no_connect (at 127 99.06))
-  (no_connect (at 127 104.14))
   (no_connect (at 152.4 99.06))
   (no_connect (at 152.4 106.68))
@@
     (stroke (width 0) (type default))
   )
+  (wire (pts (xy 142.24 66.04) (xy 142.24 68.58))
+    (stroke (width 0) (type default))
+  )
   (wire (pts (xy 218.44 54.61) (xy 214.63 54.61))
     (stroke (width 0) (type default))
@@
     (effects (font (size 1.27 1.27)) (justify right bottom))
   )
+  (label "BUTTON1" (at 127 104.14 180) (fields_autoplaced)
+    (effects (font (size 1.27 1.27)) (justify right bottom))
+  )
   (label "IGNITON_IN" (at 215.9 97.79 180) (fields_autoplaced)
     (effects (font (size 1.27 1.27)) (justify right bottom))
@@
     (effects (font (size 1.27 1.27)) (justify right bottom))
   )
-  (label "BUTTON0" (at 152.4 93.98 0) (fields_autoplaced)
-    (effects (font (size 1.27 1.27)) (justify left bottom))
-  )
   (label "BUTTON1" (at 74.93 152.4 180) (fields_autoplaced)
     (effects (font (size 1.27 1.27)) (justify right bottom))
   )
-  (label "BUTTON1" (at 152.4 96.52 0) (fields_autoplaced)
-    (effects (font (size 1.27 1.27)) (justify left bottom))
-  )
   (label "ALARM_RELAY" (at 195.58 147.32 180) (fields_autoplaced)
+    (effects (font (size 1.27 1.27)) (justify right bottom))
+  )
+  (label "BUTTON0" (at 127 101.6 180) (fields_autoplaced)
     (effects (font (size 1.27 1.27)) (justify right bottom))
   )
@@
     )
   )
-  (symbol (lib_id "power:VDD") (at 214.63 48.26 0) (unit 1)
-    (in_bom yes) (on_board yes) (dnp no) (fields_autoplaced)
-    (property "Reference" "#PWR019" (at 214.63 52.07 0)
-      (effects (font (size 1.27 1.27)) hide)
-    )
-    (property "Value" "VDD" (at 214.63 43.18 0)
-      (effects (font (size 1.27 1.27)))
-    )
-    (property "Footprint" "" (at 214.63 48.26 0)
-      (effects (font (size 1.27 1.27)) hide)
-    )
-    (property "Datasheet" "" (at 214.63 48.26 0)
-      (effects (font (size 1.27 1.27)) hide)
-    )
-    (pin "1")
-    (instances
-      (project "LTE-alarm-hw"
-        (path "/1ebed271-77ad-4435-9c3f-638c8c85758c"
-          (reference "#PWR019") (unit 1)
-        )
-      )
-    )
-  )
   (symbol (lib_id "Switch:SW_Push") (at 58.42 152.4 0) (unit 1)
     (in_bom yes) (on_board yes) (dnp no) (fields_autoplaced)
@@
     )
   )
+  (symbol (lib_id "power:+3.3V") (at 214.63 48.26 0) (unit 1)
+    (in_bom yes) (on_board yes) (dnp no) (fields_autoplaced)
+    (property "Reference" "#PWR019" (at 214.63 52.07 0)
+      (effects (font (size 1.27 1.27)) hide)
+    )
+    (property "Value" "+3.3V" (at 214.63 43.18 0)
+      (effects (font (size 1.27 1.27)))
+    )
+    (property "Footprint" "" (at 214.63 48.26 0)
+      (effects (font (size 1.27 1.27)) hide)
+    )
+    (property "Datasheet" "" (at 214.63 48.26 0)
+      (effects (font (size 1.27 1.27)) hide)
+    )
+    (pin "1")
+    (instances
+      (project "LTE-alarm-hw"
+        (path "/1ebed271-77ad-4435-9c3f-638c8c85758c"
+          (reference "#PWR019") (unit 1)
+        )
+      )
+    )
+  )
   (symbol (lib_id "power:GND") (at 195.58 149.86 0) (unit 1)
     (in_bom yes) (on_board yes) (dnp no) (fields_autoplaced)
@@
         )
       )
+    )
+  )
+  (symbol (lib_id "power:+3.3V") (at 142.24 66.04 0) (unit 1)
+    (in_bom yes) (on_board yes) (dnp no) (fields_autoplaced)
+    (property "Reference" "#PWR020" (at 142.24 69.85 0)
+      (effects (font (size 1.27 1.27)) hide)
+    )
+    (property "Value" "+3.3V" (at 142.24 60.96 0)
+      (effects (font (size 1.27 1.27)))
+    )
+    (property "Footprint" "" (at 142.24 66.04 0)
+      (effects (font (size 1.27 1.27)) hide)
+    )
+    (property "Datasheet" "" (at 142.24 66.04 0)
+      (effects (font (size 1.27 1.27)) hide)
+    )
+    (pin "1")
+    (instances
+      (project "LTE-alarm-hw"
+        (path "/1ebed271-77ad-4435-9c3f-638c8c85758c"
+          (reference "#PWR020") (unit 1)
+        )
+      )
